File: Battle_Bot_Mind/Battle_Bot_Mind.kicad_pcb (KiCad board)
At the start: 2 copper layers, 52.2 x 24.5 mm, 21 parts, among them J1 USB_C_Receptacle_USB2.0_14P, J2 Conn_01x02_Socket, J3 Conn_01x03_Pin, J4 Conn_01x01_Pin, M1 Conn_01x02_Socket, M2 Conn_01x02_Socket, U1 ESP32-C3-WROOM-02, U3 STSPIN240, U4 LD1117S33TR_SOT223

Commit message: isaac
Routing:
- net +BATT: track 49.8 -> 51.8 mm, vias 1 -> 2
- net GND: vias 16 -> 17
Changed lines of the file:
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@@
+		(net 2)
+	)
+	(via
+		(at 129.25 87.5)
+		(size 0.6)
+		(drill 0.3)
+		(layers "F.Cu" "B.Cu")
 		(net 2)
 	)
@@
 		(net 10)
 	)
-	(segment
-		(start 134 89)
-		(end 142.75 80.25)
-		(width 0.3)
-		(layer "B.Cu")
-		(net 10)
-	)
-	(segment
-		(start 128.25 89)
-		(end 134 89)
-		(width 0.3)
+	(via
+		(at 129.25 89)
+		(size 0.6)
+		(drill 0.3)
+		(layers "F.Cu" "B.Cu")
+		(net 10)
+	)
+	(segment
+		(start 140.25 83)
+		(end 134.25 89)
+		(width 0.5)
+		(layer "B.Cu")
+		(net 10)
+	)
+	(segment
+		(start 140.25 83)
+		(end 142.75 80.5)
+		(width 0.5)
+		(layer "B.Cu")
+		(net 10)
+	)
+	(segment
+		(start 142.75 80.5)
+		(end 142.75 78.75)
+		(width 0.5)
+		(layer "B.Cu")
+		(net 10)
+	)
+	(segment
+		(start 140 83.25)
+		(end 140.25 83)
+		(width 0.5)
 		(layer "B.Cu")
 		(net 10)
@@
 		(layer "B.Cu")
 		(net 10)
+	)
+	(segment
+		(start 134.25 89)
+		(end 128.25 89)
+		(width 0.5)
+		(layer "B.Cu")
+		(net 10)

Commit message: isaac
Routing:
- net /ESC_PWM: track 32.8 -> 30.5 mm, vias 1 -> 0
Changed lines of the file:
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@@
+	)
+	(segment
+		(start 148.75 74.25)
+		(end 146.999 76.001)
+		(width 0.3)
+		(layer "F.Cu")
+		(net 21)
+	)
+	(segment
+		(start 146.999 76.001)
+		(end 121.001 76.001)
+		(width 0.3)
+		(layer "F.Cu")
+		(net 21)
 	)
 	(segment
@@
 		(net 21)
 	)
-	(via
-		(at 120.5 75.5)
-		(size 0.6)
-		(drill 0.3)
-		(layers "F.Cu" "B.Cu")
+	(segment
+		(start 121.001 76.001)
+		(end 120.5 75.5)
+		(width 0.3)
+		(layer "F.Cu")
 		(net 21)
 	)
-	(segment
-		(start 135.625 76.25)
-		(end 146.75 76.25)
-		(width 0.3)
-		(layer "B.Cu")
-		(net 21)
-	)
-	(segment
-		(start 121.75 74.25)
-		(end 127 74.25)
-		(width 0.3)
-		(layer "B.Cu")
-		(net 21)
-	)
-	(segment
-		(start 128.25 73)
-		(end 132.375 73)
-		(width 0.3)
-		(layer "B.Cu")
-		(net 21)
-	)
-	(segment
-		(start 121.75 74.25)
-		(end 120.5 75.5)
-		(width 0.3)
-		(layer "B.Cu")
-		(net 21)
-	)
-	(segment
-		(start 132.375 73)
-		(end 135.625 76.25)
-		(width 0.3)
-		(layer "B.Cu")
-		(net 21)
-	)
-	(segment
-		(start 146.75 76.25)
-		(end 148.75 74.25)
-		(width 0.3)
-		(layer "B.Cu")
-		(net 21)
-	)
-	(segment
-		(start 127 74.25)
-		(end 128.25 73)
-		(width 0.3)
-		(layer "B.Cu")
-		(net 21)
-	)
