File: Battle_Bot_Mind/Battle_Bot_Mind.kicad_pcb (KiCad board)
At the start: 2 copper layers, 52.2 x 24.5 mm, 21 parts, among them J1 USB_C_Receptacle_USB2.0_14P, J2 Conn_01x02_Socket, J3 Conn_01x03_Pin, J4 Conn_01x01_Pin, M1 Conn_01x02_Socket, M2 Conn_01x02_Socket, U1 ESP32-C3-WROOM-02, U2 TB6612FNG, U4 LD1117S33TR_SOT223

Commit message: jlc
Parts:
- R3, R4: value 330r -> 300r
Changed lines of the file:
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@@
 			)
 		)
+		(property "LCSC" "C428721"
+			(at 0 0 270)
+			(unlocked yes)
+			(layer "F.Fab")
+			(hide yes)
+			(effects
+				(font
+					(size 1 1)
+					(thickness 0.15)
+				)
+			)
+		)
 		(property ki_fp_filters "Connector*:*_1x??_*")
 		(sheetname "/")
@@
 			)
 		)
+		(property "LCSC" "C2944070"
+			(at 0 0 90)
+			(unlocked yes)
+			(layer "F.Fab")
+			(hide yes)
+			(effects
+				(font
+					(size 1 1)
+					(thickness 0.15)
+				)
+			)
+		)
 		(property ki_fp_filters "ESP32?C3*WROOM?02*")
 		(sheetname "/")
@@
 			)
 		)
-		(property "Value" "330r"
+		(property "Value" "300r"
 			(at 0 1.17 90)
 			(layer "F.Fab")
@@
 			)
 		)
+		(property "LCSC" "C25102"
+			(at 0 0 90)
+			(unlocked yes)
+			(layer "F.Fab")
+			(hide yes)
+			(effects
+				(font
+					(size 1 1)
+					(thickness 0.15)
+				)
+			)
+		)
 		(property ki_fp_filters "R_*")
 		(sheetname "/")
@@
 			)
 		)
+		(property "LCSC" "C965793"
+			(at 0 0 90)
+			(unlocked yes)
+			(layer "F.Fab")
+			(hide yes)
+			(effects
+				(font
+					(size 1 1)
+					(thickness 0.15)
+				)
+			)
+		)
 		(property ki_fp_filters "LED* LED_SMD:* LED_THT:*")
 		(sheetname "/")
@@
 			)
 		)
+		(property "LCSC" "C141517"
+			(at 0 0 180)
+			(unlocked yes)
+			(layer "F.Fab")
+			(hide yes)
+			(effects
+				(font
+					(size 1 1)
+					(thickness 0.15)
+				)
+			)
+		)
 		(property ki_fp_filters "SSOP*5.3x8.2mm*P0.65mm*")
 		(sheetname "/")
@@
 			)
 		)
-		(property "Value" "330r"
+		(property "Value" "300r"
 			(at 0 1.17 90)
 			(layer "F.Fab")
@@
 			)
 		)
+		(property "LCSC" "C25102"
+			(at 0 0 90)
+			(unlocked yes)
+			(layer "F.Fab")
+			(hide yes)
+			(effects
+				(font
+					(size 1 1)
+					(thickness 0.15)
+				)
+			)
+		)
 		(property ki_fp_filters "R_*")
 		(sheetname "/")
@@
 			)
 		)
+		(property "LCSC" "C965793"
+			(at 0 0 90)
+			(unlocked yes)
+			(layer "F.Fab")
+			(hide yes)
+			(effects
+				(font
+					(size 1 1)
+					(thickness 0.15)
+				)
+			)
+		)
 		(property ki_fp_filters "LED* LED_SMD:* LED_THT:*")
 		(sheetname "/")
@@
 					(thickness 0.15)
 				)
+			)
+		)
+		(property "LCSC" "C86781"
+			(at 0 0 0)
+			(unlocked yes)
+			(layer "F.Fab")
+			(hide yes)
+			(effects
+				(font
+					(size 1 1)
+					(thickness 0.15)
+				)

Commit message: jlc2
Parts:
- M1, M2: footprint Connector_PinHeader_1.27mm:PinHeader_1x02_P1.27mm_Vertical -> Connector_PinHeader_2.54mm:PinHeader_1x02_P2.54mm_Vertical
- moved M1 1.35 mm to (138.0, 86.2), turned to -90 degrees
- moved M2 1.12 mm to (135.5, 91.0), turned to 90 degrees
Routing:
- net GND: track 27.8 -> 35.4 mm, vias 15 -> 24
- net Net-(M2-Pin_2): track 6.06 -> 8.41 mm
- net Net-(M1-Pin_1): track 6.46 -> 8.23 mm

Commit message: work
Parts:
- added M3: Conn_01x02_Socket, Connector_PinHeader_2.54mm:PinHeader_1x02_P2.54mm_Vertical, F.Cu at (122.2, 83.0)
Routing:
- net +BATT: track 74.6 -> 77.0 mm
- net GND: track 35.4 -> 37.6 mm

Commit message: work
Other:
- board text added: "100u"
Changed lines of the file:
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@@
+	)
+	(gr_line
+		(start 120.48 78.68)
+		(end 124.02 78.68)
+		(stroke
+			(width 0.1)
+			(type default)
+		)
+		(layer "B.SilkS")
 	)
 	(gr_line
@@
 	)
 	(gr_line
+		(start 124.02 78.68)
+		(end 124.02 83.75)
+		(stroke
+			(width 0.1)
+			(type default)
+		)
+		(layer "B.SilkS")
+	)
+	(gr_line
 		(start 142.35 90.77)
 		(end 142.35 92.73)
@@
 	)
 	(gr_line
+		(start 120.48 78.68)
+		(end 120.48 84.75)
+		(stroke
+			(width 0.1)
+			(type default)
+		)
+		(layer "B.SilkS")
+	)
+	(gr_line
 		(start 139.75 88)
 		(end 139.75 84.485)
@@
 		(start 142.85 90.1)
 		(end 142.85 82.9)
+		(stroke
+			(width 0.1)
+			(type default)
+		)
+		(layer "B.SilkS")
+	)
+	(gr_line
+		(start 120.5 84.75)
+		(end 122.75 84.75)
 		(stroke
 			(width 0.1)
@@
 		)
 	)
+	(gr_text "100u"
+		(at 123.75 79.25 90)
+		(layer "B.SilkS")
+		(effects
+			(font
+				(size 0.3 0.3)
+				(thickness 0.075)
+			)
+			(justify left bottom mirror)
+		)
+	)
 	(gr_text "light"
 		(at 116.25 71.72 90)
@@
 			)
 			(justify left bottom mirror)
+		)
+	)
+	(gr_text "Capacitor"
+		(at 123.75 80.5 90)
+		(layer "B.SilkS")
+		(effects
+			(font
+				(size 0.3 0.3)
+				(thickness 0.075)
+				(bold yes)
+			)
+			(justify left bottom mirror)
