File: Battle_Bot_Mind/Battle_Bot_Mind.kicad_sch (KiCad schematic)
At the start: 0 parts

Commit message: work
Parts:
- added C1, C5: 10u, Capacitor_SMD:C_0805_2012Metric, symbol Device:C
- added C6: 2.2u, Capacitor_SMD:C_0805_2012Metric, symbol Device:C
- added C9: 1n, Capacitor_SMD:C_0402_1005Metric, symbol Device:C
- added D1, D2: LED, LED_SMD:LED_0402_1005Metric, symbol Device:LED
- added DBG1, J3: Conn_01x03_Pin, Connector_PinHeader_2.00mm:PinHeader_1x03_P2.00mm_Vertical, symbol Connector:Conn_01x03_Pin
- added J1: USB_C_Receptacle_USB2.0_14P, Connector_USB:USB_C_Receptacle_HRO_TYPE-C-31-M-12, symbol Connector:USB_C_Receptacle_USB2.0_14P
- added J2: Conn_01x02_Socket, Connector_AMASS:AMASS_XT30U-F_1x02_P5.0mm_Vertical, symbol Connector:Conn_01x02_Socket
- added M1, M2: Conn_01x02_Socket, Connector_JST:JST_SH_BM02B-SRSS-TB_1x02-1MP_P1.00mm_Vertical, symbol Connector:Conn_01x02_Socket
- added R1, R2: 5.1k, Resistor_SMD:R_0402_1005Metric_Pad0.72x0.64mm_HandSolder, symbol Device:R
- added R3, R4: 300r, Resistor_SMD:R_0402_1005Metric, symbol Device:R
- added R5, R6: 22r, Resistor_SMD:R_0402_1005Metric_Pad0.72x0.64mm_HandSolder, symbol Device:R
- added R8: 20k, Resistor_SMD:R_0402_1005Metric, symbol Device:R
- added U1: ESP32-C3-WROOM-02, RF_Module:ESP32-C3-WROOM-02, symbol RF_Module:ESP32-C3-WROOM-02
- added U3: STSPIN240, Package_DFN_QFN:VQFN-16-1EP_3x3mm_P0.5mm_EP1.8x1.8mm, symbol Driver_Motor:STSPIN240
- added U4: LD1117S33TR_SOT223, Package_TO_SOT_SMD:SOT-223-3_TabPin2, symbol Regulator_Linear:LD1117S33TR_SOT223
Connections:
- new net: D1.2 (A), R4.2
- new net: M2.1 (Pin_1), U3.5 (OUTA2)
- new net: M2.2 (Pin_2), U3.3 (OUTA1)
- new net: J1.A7 (D-), J1.B7 (D-), R6.1
- new net: D2.2 (A), R3.2
- new net: J1.B5 (CC2), R2.2
- new net: J1.A5 (CC1), R1.2
- new net: J1.A6 (D+), J1.B6 (D+), R5.1
- new net: M1.1 (Pin_1), U3.10 (OUTB1)
- new net: R8.1, U3.12 (TOFF)
- new net: M1.2 (Pin_2), U3.8 (OUTB2)
- new net: DBG1.1 (Pin_1), U1.12 (IO21/TXD)
- new net: DBG1.3 (Pin_3), U1.11 (IO20/RXD)
- new net: C9.1, R8.2
- new net +3V3: C5.1, U1.1 (3V3), U1.2 (EN), U3.11 (REF), U4.2 (VO)
- new net +BATT: C6.1, J2.2 (Pin_2), J3.2 (Pin_2), U3.6 (VS), U4.3 (VI)
- new net EN: U1.4 (IO5), U3.13 (EN/FLT)
- new net ESC_PWM: J3.1 (Pin_1), U1.18 (IO0)
- new net GND: C1.2, C5.2, C6.2, C9.2, D1.1 (K), D2.1 (K), DBG1.2 (Pin_2), J1.A1 (GND), J1.A12 (GND), J1.B1 (GND), J1.B12 (GND), J1.S1 (SHIELD), J2.1 (Pin_1), J3.3 (Pin_3), R1.1, R2.1, U1.19 (GND), U1.9 (GND), U3.17 (EPAD), U3.7 (GND), U4.1 (GND)
- new net L1: R3.1, U1.15 (IO3)
- new net L2: R4.1, U1.10 (IO10)
- new net PH_A: U1.8 (IO9), U3.1 (PHA)
- new net PH_B: U1.6 (IO7), U3.15 (PHB)
- new net PWM_A: U1.3 (IO4), U3.2 (PWMA)
- new net PWM_B: U1.7 (IO8), U3.16 (PWMB)
- new net RESET: U1.5 (IO6), U3.14 (STBY/RESET)
- new net SENSE_A: U1.17 (IO1), U3.4 (SENSEA)
- new net SENSE_B: U1.16 (IO2), U3.9 (SENSEB)
- new net USB_D+: R5.2, U1.14 (IO19)
- new net USB_D-: R6.2, U1.13 (IO18)
- new net VBUS: C1.1, J1.A4 (VBUS), J1.A9 (VBUS), J1.B4 (VBUS), J1.B9 (VBUS)
Other:
- title: (none) -> BATTLE BOT BRAIN

Commit message: work
Changed lines of the file:
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@@
 		)
 	)
+	(text_box "Microcontroller"
+		(exclude_from_sim no)
+		(at 20.32 19.05 0)
+		(size 80.01 77.47)
+		(margins 0.9525 0.9525 0.9525 0.9525)
+		(stroke
+			(width 0)
+			(type solid)
+		)
+		(fill
+			(type none)
+		)
+		(effects
+			(font
+				(size 1.27 1.27)
+			)
+			(justify left top)
+		)
+	)
 	(text_box "Battery"
 		(exclude_from_sim no)
@@
 		)
 	)
-	(text_box "MOTOR DRIVERS"
+	(text_box "Brushed Speed Controller"
 		(exclude_from_sim no)
 		(at 96.52 107.95 0)
@@
 		)
 		(property "Value" "ESP32-C3-WROOM-02"
-			(at 29.972 28.448 0)
+			(at 21.082 22.86 0)
 			(effects
 				(font

Commit message: ISAAC_CHANGED_STUFF
Parts:
- removed D1: LED, LED_SMD:LED_0402_1005Metric, symbol Device:LED
- removed R4: 300r, Resistor_SMD:R_0402_1005Metric, symbol Device:R
- added J4: Conn_01x01_Pin, Connector_PinSocket_2.54mm:PinSocket_1x01_P2.54mm_Vertical, symbol Connector:Conn_01x01_Pin
Connections:
- net L2 is gone; now on net ESC_PWM: U1.10 (IO10)
- net ESC_PWM: no longer U1.18 (IO0)
- new net BOOT: J4.1 (Pin_1), U1.18 (IO0)
Changed lines of the file:
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@@
 	(text_box "Microcontroller"
 		(exclude_from_sim no)
-		(at 20.32 19.05 0)
-		(size 80.01 77.47)
+		(at 17.78 19.05 0)
+		(size 82.55 77.47)
 		(margins 0.9525 0.9525 0.9525 0.9525)
 		(stroke
@@
 	(wire
 		(pts
-			(xy 62.23 137.16) (xy 62.23 139.7)
-		)
-		(stroke
-			(width 0)
-			(type default)
-		)
-	)
-	(wire
-		(pts
 			(xy 156.21 50.8) (xy 156.21 52.07)
 		)
@@
 	(wire
 		(pts
-			(xy 40.64 137.16) (xy 49.53 137.16)
-		)
-		(stroke
-			(width 0)
-			(type default)
-		)
-	)
-	(wire
-		(pts
 			(xy 133.35 83.82) (xy 133.35 82.55)
 		)
@@
 	(wire
 		(pts
-			(xy 41.91 45.72) (xy 44.45 45.72)
+			(xy 34.29 45.72) (xy 44.45 45.72)
 		)
 		(stroke
@@
 	(wire
 		(pts
-			(xy 57.15 137.16) (xy 62.23 137.16)
-		)
-		(stroke
-			(width 0)
-			(type default)
-		)
-	)
-	(wire
-		(pts
 			(xy 129.54 157.48) (xy 130.81 157.48)
 		)
@@
 		)
 	)
-	(label "ESC_PWM"
-		(at 41.91 45.72 180)
-		(effects
-			(font
-				(size 1.27 1.27)
-			)
-			(justify right bottom)
-		)
-	)
 	(label "PH_B"
 		(at 41.91 63.5 180)
@@
 		)
 	)
-	(label "L2"
-		(at 40.64 137.16 0)
-		(effects
-			(font
-				(size 1.27 1.27)
-			)
-			(justify left bottom)
-		)
-	)
 	(label "PH_B"
 		(at 147.32 134.62 0)
@@
 		)
 	)
-	(label "L2"
-		(at 41.91 71.12 180)
+	(label "BOOT"
+		(at 41.91 45.72 180)
 		(effects
 			(font
@@
 		)
 	)
+	(label "ESC_PWM"
+		(at 41.91 71.12 180)
+		(effects
+			(font
+				(size 1.27 1.27)
+			)
+			(justify right bottom)
+		)
+	)
 	(label "USB_D+"
 		(at 163.83 76.2 270)
@@
 	)
 	(symbol
-		(lib_id "Device:R")
-		(at 53.34 137.16 90)
-		(unit 1)
-		(exclude_from_sim no)
-		(in_bom yes)
-		(on_board yes)
-		(dnp no)
-		(property "Reference" "R4"
-			(at 53.34 137.16 90)
-			(effects
-				(font
-					(size 1.27 1.27)
-				)
-			)
-		)
-		(property "Value" "300r"
-			(at 53.34 139.192 90)
-			(effects
-				(font
-					(size 1.27 1.27)
-				)
-			)
-		)
-		(property "Footprint" "Resistor_SMD:R_0402_1005Metric"
-			(at 53.34 138.938 90)
-			(effects
-				(font
-					(size 1.27 1.27)
-				)
-				(hide yes)
-			)
-		)
-		(property "Datasheet" "~"
-			(at 53.34 137.16 0)
-			(effects
-				(font
-					(size 1.27 1.27)
-				)
-				(hide yes)
-			)
-		)
-		(property "Description" ""
-			(at 53.34 137.16 0)
-			(effects
-				(font
-					(size 1.27 1.27)
-				)
-				(hide yes)
-			)
-		)
-		(pin "1"
-		)
-		(pin "2"
-		)
-		(instances
-			(project "Battle_Bot_Mind"
-				(path "/8ed2f3d0-7b52-4238-85e9-85e2bfa6cfdb"
-					(reference "R4")
-					(unit 1)
-				)
-			)
-		)
-	)
-	(symbol
 		(lib_id "power:+BATT")
 		(at 199.39 123.19 0)
@@
 	)
 	(symbol
-		(lib_id "Device:LED")
-		(at 62.23 143.51 90)
+		(lib_id "Connector:Conn_01x01_Pin")
+		(at 29.21 45.72 0)
 		(unit 1)
 		(exclude_from_sim no)
@@
 		(on_board yes)
 		(dnp no)
-		(fields_autoplaced yes)
-		(property "Reference" "D1"
-			(at 66.04 143.8274 90)
+		(property "Reference" "J4"
+			(at 33.274 40.64 0)
 			(effects
 				(font
 					(size 1.27 1.27)
 				)
-				(justify right)
 			)
 		)
-		(property "Value" "LED"
-			(at 66.04 146.3674 90)
+		(property "Value" "Conn_01x01_Pin"
+			(at 26.67 43.18 0)
 			(effects
 				(font
 					(size 1.27 1.27)
 				)
-				(justify right)
 			)
 		)
-		(property "Footprint" "LED_SMD:LED_0402_1005Metric"
-			(at 62.23 143.51 0)
+		(property "Footprint" "Connector_PinSocket_2.54mm:PinSocket_1x01_P2.54mm_Vertical"
+			(at 29.21 45.72 0)
 			(effects
 				(font
@@
 		)
 		(property "Datasheet" "~"
-			(at 62.23 143.51 0)
+			(at 29.21 45.72 0)
 			(effects
 				(font
@@
 			)
 		)
-		(property "Description" "Light emitting diode"
-			(at 62.23 143.51 0)
+		(property "Description" "Generic connector, single row, 01x01, script generated"
+			(at 29.21 45.72 0)
 			(effects
 				(font
@@
 		(pin "1"
 		)
-		(pin "2"
-		)
 		(instances
-			(project "Battle_Bot_Mind"
+			(project ""
 				(path "/8ed2f3d0-7b52-4238-85e9-85e2bfa6cfdb"
-					(reference "D1")
+					(reference "J4")
 					(unit 1)
 				)
@@
 					(unit 1)
 				)
-			)
-		)
-	)
-	(symbol
-		(lib_id "power:GND")
-		(at 62.23 147.32 0)
-		(unit 1)
-		(exclude_from_sim no)
-		(in_bom yes)
-		(on_board yes)
-		(dnp no)
-		(fields_autoplaced yes)
-		(property "Reference" "#PWR021"
-			(at 62.23 153.67 0)
-			(effects
-				(font
-					(size 1.27 1.27)
-				)
-				(hide yes)
-			)
-		)
-		(property "Value" "GND"
-			(at 62.23 152.4 0)
-			(effects
-				(font
-					(size 1.27 1.27)
-				)
-			)
-		)
-		(property "Footprint" ""
-			(at 62.23 147.32 0)
-			(effects
-				(font
-					(size 1.27 1.27)
-				)
-				(hide yes)
-			)
-		)
-		(property "Datasheet" ""
-			(at 62.23 147.32 0)
-			(effects
-				(font
-					(size 1.27 1.27)
-				)
-				(hide yes)
-			)
-		)
-		(property "Description" "Power symbol creates a global label with name \"GND\" , ground"
-			(at 62.23 147.32 0)
-			(effects
-				(font
-					(size 1.27 1.27)
-				)
-				(hide yes)
-			)
-		)
-		(pin "1"
-		)
-		(instances
-			(project "Battle_Bot_Mind"
-				(path "/8ed2f3d0-7b52-4238-85e9-85e2bfa6cfdb"
-					(reference "#PWR021")
-					(unit 1)
-				)

Commit message: work
Parts:
- J4: now not fitted; now left out of the parts list
Changed lines of the file:
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@@
 		(unit 1)
 		(exclude_from_sim no)
-		(in_bom yes)
+		(in_bom no)
 		(on_board yes)
-		(dnp no)
+		(dnp yes)
 		(property "Reference" "J4"
 			(at 33.274 40.64 0)

Commit message: work
Parts:
- DBG1: now not fitted; now left out of the parts list
Changed lines of the file:
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@@
 		(unit 1)
 		(exclude_from_sim no)
-		(in_bom yes)
+		(in_bom no)
 		(on_board yes)
-		(dnp no)
+		(dnp yes)
 		(property "Reference" "DBG1"
 			(at 94.996 41.91 0)

Commit message: work
Parts:
- removed C6: 2.2u, Capacitor_SMD:C_0805_2012Metric, symbol Device:C
- removed C9: 1n, Capacitor_SMD:C_0402_1005Metric, symbol Device:C
- removed R8: 20k, Resistor_SMD:R_0402_1005Metric, symbol Device:R
- removed U3: STSPIN240, Package_DFN_QFN:VQFN-16-1EP_3x3mm_P0.5mm_EP1.8x1.8mm, symbol Driver_Motor:STSPIN240
- added U2: TB6612FNG, Package_SO:SSOP-24_5.3x8.2mm_P0.65mm, symbol Driver_Motor:TB6612FNG
- R3: value 300r -> 330r
Connections:
- net SENSE_A is gone; now on net PWM_B: U1.17 (IO1)
- net +3V3: now also U2.20 (VCC)
- net +BATT: now also U2.13 (VM2), U2.14 (VM3), U2.24 (VM1)
- net GND: now also U2.10 (PGND2), U2.18 (GND), U2.3 (PGND1), U2.4 (PGND1), U2.9 (PGND2)
- net PWM_A: now also U2.23 (PWMA)
- net PWM_B: now also U2.15 (PWMB); no longer U1.7 (IO8)
- net at M2.1 (Pin_1): now also U2.5 (AO2), U2.6 (AO2)
- net at M2.2 (Pin_2): now also U2.1 (AO1), U2.2 (AO1)
- net at M1.1 (Pin_1): now also U2.11 (BO1), U2.12 (BO1)
- net at M1.2 (Pin_2): now also U2.7 (BO2), U2.8 (BO2)
- net EN renamed BIN2
- net BIN2: now also U2.16 (BIN2)
- net PH_A renamed AIN2
- net AIN2: now also U2.22 (AIN2)
- net PH_B renamed STBY
- net STBY: now also U2.19 (STBY)
- net RESET renamed BIN1
- net BIN1: now also U2.17 (BIN1)
- net SENSE_B: no longer names the net of U1.16 (IO2)
- new net AIN1: U1.7 (IO8), U2.21 (AIN1)
Other:
- moved on the sheet: C5, D2, R3, U4
