File: Battle_Bot_Mind/_autosave-Battle_Bot_Mind.kicad_pcb (KiCad board)
At the start: 2 copper layers, 52.2 x 24.5 mm, 19 parts, among them J1 USB_C_Receptacle_USB2.0_14P, J2 Conn_01x02_Socket, J3 Conn_01x03_Pin, J4 Conn_01x01_Pin, M1 Conn_01x02_Socket, M2 Conn_01x02_Socket, U1 ESP32-C3-WROOM-02, U2 TB6612FNG, U4 LD1117S33TR_SOT223

Commit message: work
Parts:
- added D2: LED, LED_SMD:LED_0402_1005Metric, F.Cu at (108.0, 72.3)
- added R4: 330r, Resistor_SMD:R_0402_1005Metric, F.Cu at (109.2, 72.2)
- moved J4 3.75 mm to (104.0, 72.5)
- renumbered D2 to D1
Connections:
- U1 pad 16: unconnected-(U1-IO2-Pad16) -> /L2
Routing:
- net /L2: track 0.00 -> 3.21 mm
- net /BOOT: track 3.02 -> 5.42 mm
- net Net-(D2-A): track 0.00 -> 1.27 mm
- net +BATT: track 73.5 -> 74.6 mm, vias 1 -> 2
- net GND: track 26.7 -> 27.5 mm, vias 14 -> 15
